Commit message: Setup structure
fix urdf in convert
add
pure_tf
controller
random range
xacro pi

File: src/example_description/robot/visual/my-robot.xacro (robot description, xacro)
@@ -1,4 +1,5 @@
 <?xml version="1.0"?>
 <robot xmlns:xacro="http://www.ros.org/wiki/xacro" name="example">
+    <xacro:property name="pi" value="3.14159265359" />
     <link name="link_0">
         <visual>
@@ -22,9 +23,9 @@
         <child link="link_1"/>
         <axis xyz="0.0 0.0 1.0"/>
-        <limit lower="0" upper="6.28" effort="100.0" velocity="100.0"/>
+        <limit lower="${-pi}" upper="${pi}" effort="100.0" velocity="100.0"/>
     </joint>
     <link name="link_2">
         <visual>
-            <origin rpy="3.14 0 0" xyz="0.0 0.0 0.0" />
+            <origin rpy="${pi} 0 0" xyz="0.0 0.0 0.0" />
             <geometry>
                 <mesh filename="package://example_description/meshes/link_2.stl" />
@@ -37,9 +38,9 @@
         <child link="link_2"/>
         <axis xyz="0.0 0.0 1.0"/>
-        <limit lower="0" upper="3.14" effort="100.0" velocity="100.0"/>
+        <limit lower="${-pi}" upper="${pi}" effort="100.0" velocity="100.0"/>
     </joint>
     <link name="link_3">
         <visual>
-            <origin rpy="3.14 0 0" xyz="0.0 0.0 0.0" />
+            <origin rpy="${pi} 0 0" xyz="0.0 0.0 0.0" />
             <geometry>
                 <mesh filename="package://example_description/meshes/link_3.stl" />
@@ -52,5 +53,5 @@
         <child link="link_3"/>
         <axis xyz="0.0 0.0 1.0"/>
-        <limit lower="0" upper="3.14" effort="100.0" velocity="100.0"/>
+        <limit lower="${-pi}" upper="${pi}" effort="100.0" velocity="100.0"/>
     </joint>
     <link name="end_effector">
@@ -67,5 +68,5 @@
         <child link="end_effector"/>
         <axis xyz="0.0 0.0 0.0"/>
-        <limit lower="0.0" upper="6.28" effort="100.0" velocity="100.0"/>
+        <limit lower="0.0" upper="${2*pi}" effort="100.0" velocity="100.0"/>
     </joint>
 </robot>
